File: CS4270_MODULE/CS4270_MODULE/CS4270_MODULE.kicad_sch (KiCad schematic)
At the start: 79 parts, among them J101 AudioJack3, J102 AudioJack3, J104 Conn_01x12_Pin, U101 MCP6001-OT, U102 MCP6001-OT, U103 CS4270, U104 MCP6001-OT, U105 MCP6001-OT, U106 MCP6001-OT

Commit message: finished PCB
Parts:
- removed J104: Conn_01x12_Pin, symbol Connector:Conn_01x12_Pin
- removed R103: 5R1, symbol Device:R_Small
- removed R107, R108, R109: 10k, symbol Device:R_Small
- removed R111: 0R, symbol Device:R_Small
- added H101: MountingHole, MountingHole:MountingHole_2.2mm_M2, symbol Mechanical:MountingHole
- added H102: MountingHole_Pad, MountingHole:MountingHole_2.2mm_M2_Pad_TopBottom, symbol Mechanical:MountingHole_Pad
- added H103, H104: MountingHole_Pad, MountingHole:MountingHole_2.2mm_M2_DIN965_Pad_TopBottom, symbol Mechanical:MountingHole_Pad
- added J103: Conn_01x13_Pin, Connector_PinHeader_2.54mm:PinHeader_1x13_P2.54mm_Vertical, symbol Connector:Conn_01x13_Pin
- C101, C106: footprint (none) -> Capacitor_SMD:C_0402_1005Metric; Mfr Part# (none) -> GRM155R61E105MA12D; Supplier (none) -> Mouser; Supplier Part# (none) -> 81-GRM155R61E105MA2D
- C102, C103, C104, C107, C108, C110: footprint (none) -> Capacitor_SMD:C_0402_1005Metric; Mfr Part# (none) -> C1005X7R1C104K050BC; Supplier (none) -> Mouser; Supplier Part# (none) -> 810-C1005X7R1C104K
- C105, C109, C111: footprint (none) -> Capacitor_SMD:C_0603_1608Metric; Mfr Part# (none) -> 0603ZG474ZAT2A; Supplier (none) -> Mouser; Supplier Part# (none) -> 581-0603ZG474ZAT2A
- C112, C118, C120, C121: footprint (none) -> Capacitor_SMD:C_0603_1608Metric; Mfr Part# (none) -> C0603C221G3HACTU; Supplier (none) -> Mouser; Supplier Part# (none) -> 80-C0603C221G3HACTU
- C113, C114, C116, C117, C122, C123, C126, C127: value 100n -> 100nF; footprint (none) -> Capacitor_SMD:C_0402_1005Metric; Mfr Part# (none) -> C1005X7R1C104K050BC; Supplier (none) -> Mouser; Supplier Part# (none) -> 810-C1005X7R1C104K
- C115, C119, C124, C128: footprint (none) -> Capacitor_SMD:C_0805_2012Metric; Mfr Part# (none) -> GRM21BR61C106KE15K; Supplier (none) -> Mouser; Supplier Part# (none) -> 81-GRM21BR61C106KE5K
- C125, C129: footprint (none) -> Capacitor_SMD:C_0402_1005Metric; Mfr Part# (none) -> GRM1555C1H102JA1J; Supplier (none) -> Mouser; Supplier Part# (none) -> 81-GRM1555C1H102JA1J
- D101, D102, D103, D104: footprint (none) -> footprints:SOD-323-2; Mfr Part# (none) -> PESD3V3U1UA,115; Supplier (none) -> Mouser; Supplier Part# (none) -> 771-PESD3V3U1UA-T/R
- J101, J102: footprint (none) -> footprints:JAC_TRS_3.5mm_SMD; Mfr Part# (none) -> 35RASMT2BHSNTRX; Supplier (none) -> Mouser; Supplier Part# (none) -> :502-35RASMT2BHSNTRX
- R101: footprint (none) -> Resistor_SMD:R_0603_1608Metric; Mfr Part# (none) -> ERJ-3GEYJ473V; Supplier (none) -> Mouser; Supplier Part# (none) -> 667-ERJ-3GEYJ473V
- R102: value 33R -> 22R; footprint (none) -> Resistor_SMD:R_0603_1608Metric; Mfr Part# (none) -> ERJ-PA3F22R0V; Supplier (none) -> Mouser; Supplier Part# (none) -> 667-ERJ-PA3F22R0V
- R104, R105, R106, R110, R131, R135: footprint (none) -> Resistor_SMD:R_0805_2012Metric; Mfr Part# (none) -> CR0805-JW-103ELF; Supplier (none) -> Mouser; Supplier Part# (none) -> 652-CR0805-JW-103ELF
- R112, R113, R114, R115: value 0R -> 22R; footprint (none) -> Resistor_SMD:R_0603_1608Metric; Mfr Part# (none) -> ERJ-PA3F22R0V; Supplier (none) -> Mouser; Supplier Part# (none) -> 667-ERJ-PA3F22R0V
- R116, R117, R120, R124, R125, R126, R129, R133: footprint (none) -> Resistor_SMD:R_0603_1608Metric; Mfr Part# (none) -> CR0603-FX-1001ELF; Supplier (none) -> Mouser; Supplier Part# (none) -> 652-CR0603FX-1001ELF
- R118, R119: footprint (none) -> Resistor_SMD:R_0603_1608Metric; Mfr Part# (none) -> ERJ-3GEY0R00V; Supplier (none) -> Mouser; Supplier Part# (none) -> 667-ERJ-3GEY0R00V
- R121, R122, R123, R127, R128, R132: footprint (none) -> Resistor_SMD:R_0805_2012Metric; Mfr Part# (none) -> RC0805JR-072M2L; Supplier (none) -> Mouser; Supplier Part# (none) -> 603-RC0805JR-072M2L
- R130, R134: footprint (none) -> Resistor_SMD:R_0603_1608Metric; Mfr Part# (none) -> CR0603-FX-1000ELF; Supplier (none) -> Mouser; Supplier Part# (none) -> 652-CR0603FX-1000ELF
- R136, R137: footprint (none) -> Resistor_SMD:R_0805_2012Metric; Mfr Part# (none) -> CR0805-JW-222ELF; Supplier (none) -> Mouser; Supplier Part# (none) -> 652-CR0805JW-222ELF
- U101, U102, U104, U105, U106: Mfr Part# (none) -> MCP6001UT-I/OT; Supplier (none) -> Mouser; Supplier Part# (none) -> 579-MCP6001UT-I/OT
- U103: Mfr Part# (none) -> CS4270-CZZ; Supplier (none) -> Mouser; Supplier Part# (none) -> 777-CS4270-CZZ
Connections:
- net +3V3: now also C106.1, C107.1, U103.5 (VD), J103.3 (Pin_3); no longer C110.1, R116.1, U101.5 (V+)
- net +5V: now also J103.1 (Pin_1); no longer C101.1, C102.1, R118.2, R119.1, U103.19 (VA)
- net CODEC_SDOUT: now also J103.13 (Pin_13)
- net GND: now also H102.1, H103.1, H104.1, J103.12 (Pin_12), J103.2 (Pin_2), J103.4 (Pin_4), J103.7 (Pin_7)
- net I2C_SCL: now also J103.5 (Pin_5)
- net I2C_SDA: now also J103.6 (Pin_6)
- net I2S_BCLK: now also J103.8 (Pin_8)
- net I2S_MCLK: now also J103.9 (Pin_9)
- net I2S_SDIN: now also J103.11 (Pin_11)
- net I2S_WSCLK: now also J103.10 (Pin_10)
- net L_FILT_CODEC: no longer C115.1, C118.1, R126.1
- net R_FILT_CODEC: no longer C119.1, C121.1, R125.1
- new net L_FILT_CODEC_MIC: C115.1, C118.1, R126.1
- new net R_FILT_CODEC_MIC: C119.1, C121.1, R125.1
- new net VCC: C101.1, C102.1, C110.1, R116.1, R118.2, R119.1, U101.5 (V+), U103.19 (VA)
Other:
- note added: "Mounting holes"
- note removed: "Note: Put the 103 resistor in case VD is using the same supply of VA Put the R111 resistor in case VD is using another supply"
- moved on the sheet: R118, R119
