File: CS4270_MODULE/CS4270_MODULE/CS4270_MODULE.kicad_pcb (KiCad board)
At the start: 4 copper layers, 54.5 x 38 mm, 81 parts, among them J101 AudioJack3, J102 AudioJack3, J103 Conn_01x13_Pin, U101 MCP6001-OT, U102 MCP6001-OT, U103 CS4270, U104 MCP6001-OT, U105 MCP6001-OT, U106 MCP6001-OT

Commit message: .
Parts:
- moved H102 3.70 mm to (177.3, 79.0)
- moved R136 3.35 mm to (179.4, 60.8)
- moved R137 3.35 mm to (179.4, 57.2)
- moved J103 2.50 mm to (185.5, 47.3)
- moved R118 2.21 mm to (180.8, 50.4)
- moved R119 2.21 mm to (180.8, 48.8)
- moved R102 1.30 mm to (182.2, 76.5)
- moved R110 1.15 mm to (177.6, 51.2)
Routing:
- net GND: track 39.4 -> 28.3 mm, vias 116 -> 121
- net +3V3: track 82.3 -> 76.4 mm
- net /CODEC_SDOUT: track 6.73 -> 3.01 mm
- net /I2C_SDA: track 18.6 -> 15.8 mm
- net /I2C_SCL: track 19.2 -> 16.6 mm
- net /I2S_WSCLK: track 13.3 -> 10.8 mm
- net /I2S_SDIN: track 13.8 -> 11.3 mm
- net /I2S_MCLK: track 13.2 -> 10.7 mm
- net /I2S_BCLK: track 13.6 -> 11.1 mm
- net VCC: track 51.5 -> 49.3 mm
- net /CODEC_RST: track 17.5 -> 16.3 mm
- net /R_CODEC_IN: track 17.0 -> 16.3 mm
- net +5V: track 5.62 -> 4.97 mm
- net /CODEC_SDOUT_R: track 22.9 -> 23.5 mm
Other:
- board size 54.5 x 38 mm -> 51.6 x 38 mm
